File: board/board.kicad_pcb (KiCad board)
At the start: 2 copper layers, 21 x 13 mm, 1 part

Commit message: initial
Parts:
- removed LOGO1: Logo_Open_Hardware_Small, Symbol:OSHW-Symbol_6.7x6mm_SilkScreen
- added C1: 100nF, Capacitor_SMD:C_0603_1608Metric, F.Cu at (83.9, 82.5)
- added C3: 1uF, Capacitor_SMD:C_0603_1608Metric, F.Cu at (90.0, 77.5)
- added J1: 001_I2C, on_edge:on_edge_2x05_device, F.Cu at (77.0, 80.5)
- added J2: 001_I2C, on_edge:on_edge_2x05_host, F.Cu at (98.0, 80.5)
- added R1: 0R, Resistor_SMD:R_0603_1608Metric, F.Cu at (84.2, 78.0)
- added R2: 0R, Resistor_SMD:R_0603_1608Metric, F.Cu at (92.0, 78.5)
- added U1: SHT30-DIS, Sensor_Humidity:Sensirion_DFN-8-1EP_2.5x2.5mm_P0.5mm_EP1.1x1.7mm, F.Cu at (87.5, 77.5)
Routing:
- net GND: track 0.00 -> 30.5 mm, vias 0 -> 2
- net Net-(J1-Pad5): track 0.00 -> 26.2 mm, vias 0 -> 4
- net +3.3V: track 0.00 -> 23.7 mm, vias 0 -> 4
- net /sensor/SDA: track 0.00 -> 22.6 mm
- net /sensor/SCL: track 0.00 -> 19.3 mm, vias 0 -> 2
- net Net-(J1-Pad8): track 0.00 -> 18.9 mm, vias 0 -> 1
- net Net-(J1-Pad4): track 0.00 -> 18.4 mm
- net +5V: track 0.00 -> 16.9 mm
- net /sensor/~{reset}: track 0.00 -> 3.44 mm
- net /sensor/int: track 0.00 -> 1.43 mm
Other:
- outline, holes or cut-outs redrawn
- rule pad_to_mask_clearance: 0 -> 0.04
- board text added: "osf.001"
- board text added: "osf.b088.v1.0"
