File: board/sensor.kicad_sch (KiCad schematic)
At the start: 2 parts, among them U1 SHT30-DIS

Commit message: used new normal rounded corners and added ground planes
Parts:
- U1: Digi-Key_PN (none) -> 1649-SHT30-DIS-B10KSCT-ND; MPN (none) -> SHT30-DIS-B10KS
Changed lines of the file:
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@@
+      (effects (font (size 1.27 1.27)) hide)
+    )
+    (property "MPN" "SHT30-DIS-B10KS" (id 4) (at 130.175 96.52 0)
+      (effects (font (size 1.27 1.27)) hide)
+    )
+    (property "Digi-Key_PN" "1649-SHT30-DIS-B10KSCT-ND" (id 5) (at 130.175 96.52 0)
       (effects (font (size 1.27 1.27)) hide)
     )

Commit message: added LCSC part numbers
Parts:
- C1: lcsc (none) -> C14663
- U1: lcsc (none) -> C77361
